File: Solar Cell offgrid Power.kicad_pcb (KiCad board)
At the start: 2 copper layers, 139.2 x 125.1 mm, 25 parts, among them J1 Conn_01x10_Socket, J2 Conn_01x10_Pin, J3 Screw_Terminal_01x02

Commit message: Add files via upload
Parts:
- added ?: , , F.Cu at (92.3, 59.4)
- added REF**: TestPoint_Pad_4.0x4.0mm, TestPoint:TestPoint_Pad_4.0x4.0mm, F.Cu at (221.2, 101.3)
- added REF**: TestPoint_Pad_4.0x4.0mm, TestPoint:TestPoint_Pad_4.0x4.0mm, F.Cu at (92.2, 101.2)
- added REF**: TestPoint_Pad_4.0x4.0mm, TestPoint:TestPoint_Pad_4.0x4.0mm, F.Cu at (221.3, 90.9)
- added REF**: TestPoint_Pad_4.0x4.0mm, TestPoint:TestPoint_Pad_4.0x4.0mm, F.Cu at (92.3, 81.0)
- added REF**: TestPoint_Pad_4.0x4.0mm, TestPoint:TestPoint_Pad_4.0x4.0mm, F.Cu at (92.2, 91.1)
- added REF**: TestPoint_Pad_4.0x4.0mm, TestPoint:TestPoint_Pad_4.0x4.0mm, F.Cu at (221.2, 80.8)
- moved G*** 55.4 mm to (105.4, 142.9)
- moved REF** 23.5 mm to (183.0, 141.7)
- moved G*** 6.65 mm to (105.5, 148.3)
- moved REF** 5.44 mm to (202.3, 141.2)
- moved J3 3.16 mm to (90.5, 50.4)
- moved J2 2.45 mm to (91.2, 102.5)
Connections:
- J3 pad 2: PWR_HOME -> PWR
Routing:
- net GND: track 408.9 -> 442.9 mm
- net PWR: track 314.5 -> 288.2 mm, vias 24 -> 36
- net PWR_HOME: track 10.6 -> 0.00 mm
- net (no net): vias 12 -> 0
Other:
- board size 139.2 x 125.1 mm -> 144.5 x 125.1 mm
- board text added: "For a Single Monocrystalline Blue Solar Tile TDB125 Series or Parallel Connectivity 125x125mm"
- board text added: "REV. 04-2023"
- board text removed: "FOR A SINGLE Monocrystalline Blue Solar Tile TDB125 Series or Parallel Connectivity 125x125mm"
- board text removed: "REV. 03-2023"
